Commit message: update sensors

File: simulator/src/simulator/otter_gazebo/urdf/sensors/otter_lidar.xacro (robot description, xacro)
@@ -6,5 +6,5 @@
         <origin xyz="0 0 -0.05"/>
         <geometry>
-          <cylinder radius="0.025" length="0.1" />
+          <cylinder radius="0" length="0" />
         </geometry>
         <material name="${name}_visual_material">
@@ -25,4 +25,5 @@
           <scan>
             <horizontal>
+              <!-- 720, 1, -3.14, 3.14 -->
               <samples>720</samples>
               <resolution>1</resolution>
@@ -36,6 +37,6 @@
             <!-- Maximum distance of the beam -->
             <max>${max_range}</max>
-            <!-- Linear resolution of the beam -->
-            <resolution>0.02</resolution>
+            <!-- Linear resolution of the beam 0.02 -->
+            <resolution>0.5</resolution>
           </range>
         </ray>

File: simulator/src/simulator/usv_worlds/worlds/usv.world.xacro (robot description, xacro)
@@ -24,5 +24,5 @@
     <gui fullscreen='0'>
       <camera name='user_camera'>
-        <pose frame=''>-9.35 -10.43 2.92 0 0.27 0.40</pose>
+        <pose frame=''>50 -15 15 0 0.35 2.75</pose>
         <view_controller>orbit</view_controller>
       </camera>
